Commit message: update damping and i

File: sr_description/arm/xacro/hand_support/shadowarm_handsupport_motor.urdf.xacro (robot description, xacro)
@@ -6,5 +6,5 @@
 	<origin xyz="0 0 0" rpy="0 0 0" />
 	<mass value="0.75" />
-	<inertia  ixx="0.001" ixy="0.0"  ixz="0.0"  iyy="0.001"  iyz="0.0"  izz="0.001" />
+	<inertia  ixx="0.0001" ixy="0.0"  ixz="0.0"  iyy="0.0001"  iyz="0.0"  izz="0.0001" />
       </inertial>
       <visual>
@@ -35,4 +35,8 @@
       <dynamics damping="30.0"/>
     </joint>
+    <gazebo reference="ElbowJRotate">
+      <provideFeedback>1</provideFeedback>
+      <implicitSpringDamper>1</implicitSpringDamper>
+    </gazebo>
     <xacro:shadowarm_handsupport_motor_transmission />
   </xacro:macro>

File: sr_description/arm/xacro/lower_arm/shadowarm_lowerarm.urdf.xacro (robot description, xacro)
@@ -6,6 +6,6 @@
 	<origin xyz="0 0 0" rpy="0 0 0" />
 	<mass value="0.5" />
-	<inertia  ixx="0.001" ixy="0.0"  ixz="0.0"  iyy="0.001"  iyz="0.0"
-	izz="0.001" />
+	<inertia  ixx="0.0001" ixy="0.0"  ixz="0.0"  iyy="0.0001"  iyz="0.0"
+	izz="0.0001" />
       </inertial>
       <visual>
@@ -35,4 +35,8 @@
       <dynamics damping="20.0"/>
     </joint>
+    <gazebo reference="ElbowJSwing">
+      <provideFeedback>1</provideFeedback>
+      <implicitSpringDamper>1</implicitSpringDamper>
+    </gazebo>
     <xacro:shadowarm_lowerarm_transmission />
   </xacro:macro>

File: sr_description/arm/xacro/trunk/shadowarm_trunk.urdf.xacro (robot description, xacro)
@@ -35,4 +35,8 @@
       <dynamics damping="30.0"/>
     </joint>
+    <gazebo reference="ShoulderJRotate">
+      <provideFeedback>1</provideFeedback>
+      <implicitSpringDamper>1</implicitSpringDamper>
+    </gazebo>
     <xacro:shadowarm_trunk_transmission />
   </xacro:macro>

File: sr_description/arm/xacro/upper_arm/shadowarm_upperarm.urdf.xacro (robot description, xacro)
@@ -6,5 +6,5 @@
         <origin xyz="0 0 0.0" rpy="0 0 0" />
         <mass value="0.5" />
-        <inertia  ixx="0.001" ixy="0.0"  ixz="0.0"  iyy="0.001"  iyz="0.0" izz="0.001" />
+        <inertia  ixx="0.0001" ixy="0.0"  ixz="0.0"  iyy="0.0001"  iyz="0.0" izz="0.0001" />
       </inertial>
       <visual>
@@ -34,4 +34,8 @@
       <dynamics damping="30.0"/>
     </joint>
+    <gazebo reference="ShoulderJSwing">
+      <provideFeedback>1</provideFeedback>
+      <implicitSpringDamper>1</implicitSpringDamper>
+    </gazebo>
     <xacro:shadowarm_upperarm_transmission />
   </xacro:macro>

File: sr_description/hand/xacro/finger/biotac/biotac.urdf.xacro (robot description, xacro)
@@ -53,4 +53,8 @@
       <dynamics damping="10.0"/>
     </joint>
+    <gazebo reference="${joint_prefix}J2">
+      <provideFeedback>1</provideFeedback>
+      <implicitSpringDamper>1</implicitSpringDamper>
+    </gazebo>
     <link name="${link_prefix}_J1_dummy">
       <inertial>
@@ -68,4 +72,8 @@
       <dynamics damping="10.0"/>
     </joint>
+    <gazebo reference="${joint_prefix}J1">
+    <provideFeedback>1</provideFeedback>
+    <implicitSpringDamper>1</implicitSpringDamper>
+    </gazebo>
     <xacro:middle_transmission />
     <link name="${link_prefix}biotac">

File: sr_description/hand/xacro/finger/biotac/edc_muscle_biotac.urdf.xacro (robot description, xacro)
@@ -53,4 +53,8 @@
       <dynamics damping="10.0"/>
     </joint>
+    <gazebo reference="${joint_prefix}J2">
+    <provideFeedback>1</provideFeedback>
+    <implicitSpringDamper>1</implicitSpringDamper>
+    </gazebo>
     <link name="${link_prefix}_J1_dummy">
       <inertial>
@@ -68,4 +72,8 @@
       <dynamics damping="10.0"/>
     </joint>
+    <gazebo reference="${joint_prefix}J1">
+    <provideFeedback>1</provideFeedback>
+    <implicitSpringDamper>1</implicitSpringDamper>
+    </gazebo>
     <xacro:middle_transmission />
     <link name="${link_prefix}biotac">

File: sr_description/hand/xacro/finger/distal/distal.urdf.xacro (robot description, xacro)
@@ -55,4 +55,8 @@
       <dynamics damping="10.0"/>
     </joint>
+    <gazebo reference="${joint_prefix}J1">
+    <provideFeedback>1</provideFeedback>
+    <implicitSpringDamper>1</implicitSpringDamper>
+    </gazebo>
     <link name="${link_prefix}tip">
       <inertial>

File: sr_description/hand/xacro/finger/distal/distal_biotac.urdf.xacro (robot description, xacro)
@@ -55,4 +55,8 @@
       <dynamics damping="10.0"/>
     </joint>
+    <gazebo reference="${joint_prefix}J1">
+    <provideFeedback>1</provideFeedback>
+    <implicitSpringDamper>1</implicitSpringDamper>
+    </gazebo>
 <!--
     <xacro:distal_transmission />

File: sr_description/hand/xacro/finger/distal/distal_ellipsoid.urdf.xacro (robot description, xacro)
@@ -61,4 +61,8 @@
       <dynamics damping="10.0"/>
     </joint>
+    <gazebo reference="${joint_prefix}J1">
+    <provideFeedback>1</provideFeedback>
+    <implicitSpringDamper>1</implicitSpringDamper>
+    </gazebo>
     <link name="${link_prefix}tip">
       <inertial>

File: sr_description/hand/xacro/finger/knuckle/edc_muscle_knuckle.urdf.xacro (robot description, xacro)
@@ -56,4 +56,8 @@
       <dynamics damping="10.0"/>
     </joint>
+    <gazebo reference="${joint_prefix}J4">
+    <provideFeedback>1</provideFeedback>
+    <implicitSpringDamper>1</implicitSpringDamper>
+    </gazebo>
     <xacro:knuckle_transmission />
   </xacro:macro>

File: sr_description/hand/xacro/finger/knuckle/knuckle.urdf.xacro (robot description, xacro)
@@ -13,6 +13,6 @@
 	<!--<insert_block name="origin" /> -->
 	<mass value="0.008" />
-	<inertia  ixx="0.00001" ixy="0.0"  ixz="0.0"  iyy="0.00001"  iyz="0.0"
-	izz="0.00001" />
+	<inertia  ixx="1e-6" ixy="0.0"  ixz="0.0"  iyy="1e-6"  iyz="0.0"
+	izz="1e-6" />
       </inertial>
       <visual>
@@ -56,4 +56,8 @@
       <dynamics damping="10.0"/>
     </joint>
+    <gazebo reference="${joint_prefix}J4">
+    <provideFeedback>1</provideFeedback>
+    <implicitSpringDamper>1</implicitSpringDamper>
+    </gazebo>
     <xacro:knuckle_transmission />
   </xacro:macro>

File: sr_description/hand/xacro/finger/lfmetacarpal/edc_muscle_lfmetacarpal.urdf.xacro (robot description, xacro)
@@ -63,4 +63,8 @@
       <dynamics damping="10.0"/>
     </joint>
+    <gazebo reference="LFJ5">
+    <provideFeedback>1</provideFeedback>
+    <implicitSpringDamper>1</implicitSpringDamper>
+    </gazebo>
     <xacro:lfmetacarpal_transmission />
   </xacro:macro>

File: sr_description/hand/xacro/finger/lfmetacarpal/lfmetacarpal.urdf.xacro (robot description, xacro)
@@ -22,5 +22,5 @@
         <origin xyz="0 0 0.04" rpy="0 0 0" />
 	    <mass value="0.075" />
-	    <inertia  ixx="0.1" ixy="0.0"  ixz="0.0"  iyy="0.1"  iyz="0.0" izz="0.1" />
+	    <inertia  ixx="1e-6" ixy="0.0"  ixz="0.0"  iyy="1e-6"  iyz="0.0" izz="1e-6" />
       </inertial>
       <visual>
@@ -63,4 +63,8 @@
       <dynamics damping="10.0"/>
     </joint>
+    <gazebo reference="LFJ5">
+    <provideFeedback>1</provideFeedback>
+    <implicitSpringDamper>1</implicitSpringDamper>
+    </gazebo>
     <xacro:lfmetacarpal_transmission />
   </xacro:macro>

File: sr_description/hand/xacro/finger/little_finger_ellipsoid.urdf.xacro (robot description, xacro)
@@ -60,4 +60,8 @@
       <dynamics damping="10.0"/>
     </joint>
+    <gazebo reference="LFJ4">
+      <provideFeedback>1</provideFeedback>
+      <implicitSpringDamper>1</implicitSpringDamper>
+    </gazebo>
     <transmission type="sr_mechanism_model/SimpleTransmission" name="lfknuckle_transmission">
       <actuator name="LFJ4" />

File: sr_description/hand/xacro/finger/middle/middle.urdf.xacro (robot description, xacro)
@@ -54,4 +54,8 @@
       <dynamics damping="10.0"/>
     </joint>
+    <gazebo reference="${joint_prefix}J2">
+    <provideFeedback>1</provideFeedback>
+    <implicitSpringDamper>1</implicitSpringDamper>
+    </gazebo>
     <xacro:middle_transmission />
   </xacro:macro>

File: sr_description/hand/xacro/finger/proximal/edc_muscle_proximal.urdf.xacro (robot description, xacro)
@@ -54,4 +54,8 @@
       <dynamics damping="10.0"/>
     </joint>
+    <gazebo reference="${joint_prefix}J3">
+    <provideFeedback>1</provideFeedback>
+    <implicitSpringDamper>1</implicitSpringDamper>
+    </gazebo>
     <xacro:proximal_transmission />
   </xacro:macro>

File: sr_description/hand/xacro/finger/proximal/proximal.urdf.xacro (robot description, xacro)
@@ -54,4 +54,8 @@
       <dynamics damping="10.0"/>
     </joint>
+    <gazebo reference="${joint_prefix}J3">
+      <provideFeedback>1</provideFeedback>
+      <implicitSpringDamper>1</implicitSpringDamper>
+    </gazebo>
     <xacro:proximal_transmission />
   </xacro:macro>

File: sr_description/hand/xacro/forearm/forearm_motor.urdf.xacro (robot description, xacro)
@@ -6,5 +6,5 @@
 	<origin xyz="0 0 0.09" rpy="0 0 0"/>
 	<mass value="3.0" />
-	<inertia  ixx="1.0" ixy="0.0"  ixz="0.0"  iyy="1.0"  iyz="0.0"  izz="1.0" />
+	<inertia  ixx="0.001" ixy="0.0"  ixz="0.0"  iyy="0.001"  iyz="0.0"  izz="0.001" />
       </inertial>
       <visual>

File: sr_description/hand/xacro/palm/edc_muscle_palm.urdf.xacro (robot description, xacro)
@@ -63,4 +63,8 @@
       <dynamics damping="30.0"/>
     </joint>
+    <gazebo reference="WRJ1">
+      <provideFeedback>1</provideFeedback>
+      <implicitSpringDamper>1</implicitSpringDamper>
+    </gazebo>
     <xacro:shadowhand_palm_transmission />
   </xacro:macro>

File: sr_description/hand/xacro/palm/palm.urdf.xacro (robot description, xacro)
@@ -22,5 +22,5 @@
 	<origin xyz="0 0 0.035" rpy="0 0 0" />
 	<mass value="0.3" />
-	<inertia  ixx="0.5" ixy="0.0"  ixz="0.0"  iyy="0.5"  iyz="0.0"	izz="0.3" />
+	<inertia  ixx="0.0005" ixy="0.0"  ixz="0.0"  iyy="0.0005"  iyz="0.0"	izz="0.0003" />
       </inertial>
       <visual>
@@ -63,4 +63,8 @@
       <dynamics damping="30.0"/>
     </joint>
+    <gazebo reference="WRJ1">
+      <provideFeedback>1</provideFeedback>
+      <implicitSpringDamper>1</implicitSpringDamper>
+    </gazebo>
     <xacro:shadowhand_palm_transmission />
   </xacro:macro>
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