Commit message: add forearm + hand only model.  add expanded urdf and sdf files.

File: sr_description/model_arm_and_hand.urdf (robot description, URDF)
Before this commit: robot shadowhand_motor, 30 links, 29 joints
Links:
- added link shadowarm_base, mass 0.4; collision mesh filename=package://sr_description/arm/model/arm_base.dae scale=0.001 0.001 0.001; visual mesh filename=package://sr_description/arm/model/arm_base.dae scale=0.001 0.001 0.001
- added link shadowarm_handsupport, mass 0.75; collision cylinder length=0.001 radius=0.06; visual mesh filename=package://sr_description/arm/model/elbow_rotate_motor.dae scale=0.001 0.001 0.001
- added link shadowarm_lowerarm, mass 0.5; collision mesh filename=package://sr_description/arm/model/elbow_flex.dae scale=0.001 0.001 0.001; visual mesh filename=package://sr_description/arm/model/elbow_flex.dae scale=0.001 0.001 0.001
- added link shadowarm_trunk, mass 0.5; collision mesh filename=package://sr_description/arm/model/arm_trunk.dae scale=0.001 0.001 0.001; visual mesh filename=package://sr_description/arm/model/arm_trunk.dae scale=0.001 0.001 0.001
- added link shadowarm_upperarm, mass 0.5; collision mesh filename=package://sr_description/arm/model/upper_arm.dae scale=0.001 0.001 0.001; visual mesh filename=package://sr_description/arm/model/upper_arm.dae scale=0.001 0.001 0.001
- added link world
Joints:
- added joint ElbowJRotate: type revolute, parent shadowarm_lowerarm, child shadowarm_handsupport, origin xyz=0.08 0 0.125 rpy=0.0 0 0, axis 0 0 -1, limit lower=-1.57079632679 upper=1.57079632679 effort=1000.0 velocity=10.0
- added joint ElbowJSwing: type revolute, parent shadowarm_upperarm, child shadowarm_lowerarm, origin xyz=0 0 0.369 rpy=0 0 0, axis 0 -1 0, limit lower=0.52 upper=2.09439510239 effort=1000.0 velocity=10.0
- added joint ShoulderJRotate: type revolute, parent shadowarm_base, child shadowarm_trunk, origin xyz=0 0 0.01 rpy=0.0 0.0 0.0, axis 0 0 1, limit lower=-0.785398163397 upper=1.57079632679 effort=1000.0 velocity=10.0
- added joint ShoulderJSwing: type revolute, parent shadowarm_trunk, child shadowarm_upperarm, origin xyz=0 -0.134 0.5305 rpy=0 -3.14159265359 0.0, axis 0 -1 0, limit lower=0 upper=1.57079632679 effort=1000.0 velocity=10.0
- added joint arm_link: type fixed, parent shadowarm_handsupport, child forearm, origin xyz=0 0 0 rpy=0 0 2.35619449
- added joint arm_to_world_fixed: type fixed, parent world, child shadowarm_base, origin xyz=0 -1 1.0 rpy=0 0 0

File: sr_description/model_forearm_and_hand.urdf (robot description, URDF)
Before this commit: robot arm_and_hand, 36 links, 35 joints
Links:
- removed link shadowarm_base
- removed link shadowarm_lowerarm
- removed link shadowarm_trunk
- removed link shadowarm_upperarm
Joints:
- removed joint ElbowJSwing
- removed joint ShoulderJRotate
- removed joint ShoulderJSwing
- removed joint arm_to_world_fixed
- joint ElbowJRotate: parent shadowarm_lowerarm -> world
- joint arm_link: origin xyz=0 0 0 rpy=0 0 2.35619449 -> xyz=0 0 1.2 rpy=1.57 3.14 1.57
