Commit message: update model, adding version from handsupport and up, and update forearm and hand model so it includes the elbow.

File: sr_description/model_handsupport_and_hand.urdf (robot description, URDF)
Before this commit: robot arm_and_hand, 33 links, 32 joints
Links:
- removed link shadowarm_lowerarm
Joints:
- removed joint ElbowJSwing
- joint ElbowJRotate: parent shadowarm_lowerarm -> world
- joint arm_link: origin xyz=0.08 0 0.121 rpy=0 0 2.35619449 -> xyz=0 0 1.2 rpy=1.57 3.14 1.57; parent shadowarm_lowerarm -> shadowarm_handsupport

File: sr_description/robots/forearm_and_hand_motor.urdf.xacro (robot description, xacro)
@@ -3,12 +3,26 @@
   <xacro:include filename="$(find sr_description)/hand/xacro/full_hand_motor.urdf.xacro" />
   <xacro:include filename="$(find sr_description)/other/xacro/gazebo/gazebo.urdf.xacro" />
+<!--
+  <xacro:include filename="$(find sr_description)/arm/xacro/full_arm_motor.urdf.xacro" />
+-->
+  <xacro:include filename="$(find sr_description)/arm/xacro/lower_arm/shadowarm_lowerarm.urdf.xacro" />
   <xacro:include filename="$(find sr_description)/arm/xacro/hand_support/shadowarm_handsupport_motor.urdf.xacro" />
   <link name="world" />
-  <xacro:shadowarm_handsupport_motor parent="world">
+  <!--
+  <joint name="arm_to_world_fixed" type="fixed">
+    <parent link="world"/>
+    <child link="shadowarm_lowerarm"/>
+    <origin xyz="0 0 1.2" rpy="${1.57} ${3.14} ${1.57}" />
+  </joint>
+  -->
+  <xacro:shadowarm_lowerarm parent="world">
+  </xacro:shadowarm_lowerarm>
+  <xacro:shadowarm_handsupport_motor parent="shadowarm_lowerarm">
   </xacro:shadowarm_handsupport_motor>
+  <!-- connects forearm to lowerarm -->
   <joint name="arm_link" type="fixed">
-    <parent link="shadowarm_handsupport"/>
+    <parent link="shadowarm_lowerarm"/>
     <child link="forearm"/>
-    <origin xyz="0 0 1.2" rpy="${1.57} ${3.14} ${1.57}" />
+    <origin xyz="0.08 0 0.121" rpy="0 0 ${2.35619449}" />
   </joint>
   <xacro:shadowhand_motor>
