Commit message: Fix model_forearm_and_hand.urdf and its converted sdf

File: sr_description/model_forearm_and_hand.urdf (robot description, URDF)
Before this commit: robot arm_and_hand, 33 links, 32 joints
Joints:
- joint arm_link: parent shadowarm_lowerarm -> shadowarm_handsupport

Commit message: Fix link positions by: Clean copy and modify model_forearm_and_hand.urdf from model_arm_and_hand.urdf, and generate model_forearm_and_hand.sdf from it

File: sr_description/model_forearm_and_hand.urdf (robot description, URDF)
Before this commit: robot arm_and_hand, 33 links, 32 joints
Joints:
- joint arm_link: origin xyz=0.08 0 0.121 rpy=0 0 2.35619449 -> xyz=0 0 0 rpy=0 0 2.35619449

Commit message: Restore mass and inertia

File: sr_description/model_forearm_and_hand.urdf (robot description, URDF)
Before this commit: robot arm_and_hand, 33 links, 32 joints
Links:
- link shadowarm_handsupport: mass 0.75 -> 3.75
- link shadowarm_lowerarm: mass 0.5 -> 3.5

Commit message: Restore all the mass and inertia to the before this pull request

File: sr_description/model_forearm_and_hand.urdf (robot description, URDF)
Before this commit: robot arm_and_hand, 33 links, 32 joints
Links:
- link shadowarm_handsupport: mass 3.75 -> 0.75
- link shadowarm_lowerarm: mass 3.5 -> 0.5
Joints:
- joint arm_link: origin xyz=0 0 0 rpy=0 0 2.35619449 -> xyz=0.08 0 0.121 rpy=0 0 2.35619449
