Commit message: update inertia values to match finger collision geometries

File: sr_description/hand/xacro/finger/distal/distal.urdf.xacro (robot description, xacro)
@@ -12,6 +12,7 @@
 	<mass value="0.010" />
 	<origin xyz="0 0 0.013" />
-	<inertia  ixx="0.00001" ixy="0.0"  ixz="0.0"  iyy="0.00001"  iyz="0.0"
-	izz="0.00001" />
+	<inertia  ixx="0.0000001" ixy="0.0"  ixz="0.0"
+            iyy="0.0000001"  iyz="0.0"
+            izz="0.0000001" />
       </inertial>
       <visual>

File: sr_description/hand/xacro/finger/knuckle/knuckle.urdf.xacro (robot description, xacro)
@@ -13,6 +13,7 @@
 	<!--<insert_block name="origin" /> -->
 	<mass value="0.008" />
-	<inertia  ixx="1e-6" ixy="0.0"  ixz="0.0"  iyy="1e-6"  iyz="0.0"
-	izz="1e-6" />
+	<inertia  ixx="0.0000002" ixy="0.0"  ixz="0.0"
+            iyy="0.0000002" iyz="0.0"
+            izz="0.0000002" />
       </inertial>
       <visual>

File: sr_description/hand/xacro/finger/lfmetacarpal/lfmetacarpal.urdf.xacro (robot description, xacro)
@@ -22,5 +22,7 @@
         <origin xyz="0 0 0.04" rpy="0 0 0" />
 	    <mass value="0.075" />
-	    <inertia  ixx="1e-6" ixy="0.0"  ixz="0.0"  iyy="1e-6"  iyz="0.0" izz="1e-6" />
+	    <inertia  ixx="5e-6" ixy="0.0"  ixz="0.0"
+                iyy="5e-6"  iyz="0.0"
+                izz="3e-6" />
       </inertial>
       <visual>

File: sr_description/hand/xacro/finger/middle/middle.urdf.xacro (robot description, xacro)
@@ -12,6 +12,7 @@
 	<origin xyz="0 0 0.0125" rpy="0 0 0" />
 	<mass value="0.012" />
-	<inertia  ixx="0.0001" ixy="0.0"  ixz="0.0"  iyy="0.0001"  iyz="0.0"
-	izz="0.00001" />
+	<inertia  ixx="0.0000008" ixy="0.0"  ixz="0.0"
+            iyy="0.0000008" iyz="0.0"
+            izz="0.0000003" />
       </inertial>
       <visual>

File: sr_description/hand/xacro/finger/proximal/proximal.urdf.xacro (robot description, xacro)
@@ -12,6 +12,7 @@
 	<mass value="0.014" />
 	<origin xyz="0 0 0.0225" />
-	<inertia  ixx="0.00001" ixy="0.0"  ixz="0.0"  iyy="0.00001"  iyz="0.0"
-	izz="0.00001" />
+	<inertia  ixx="0.0000010" ixy="0.0"  ixz="0.0"
+            iyy="0.0000010" iyz="0.0"
+            izz="0.0000005" />
       </inertial>
       <visual>

File: sr_description/hand/xacro/palm/palm.urdf.xacro (robot description, xacro)
@@ -22,5 +22,7 @@
 	<origin xyz="0 0 0.035" rpy="0 0 0" />
 	<mass value="0.3" />
-	<inertia  ixx="0.0005" ixy="0.0"  ixz="0.0"  iyy="0.0005"  iyz="0.0"	izz="0.0003" />
+	<inertia  ixx="0.0001" ixy="0.0"  ixz="0.0"
+            iyy="0.0002" iyz="0.0"
+          	izz="0.0001" />
       </inertial>
       <visual>

File: sr_description/hand/xacro/thumb/thbase.urdf.xacro (robot description, xacro)
@@ -22,6 +22,7 @@
 	<mass value="0.010" />
 	  <origin xyz="0 0 0" rpy="0 0 0"/>
-	<inertia  ixx="0.00001" ixy="0.0"  ixz="0.0"  iyy="0.00001"  iyz="0.0"
-	izz="0.00001" />
+	<inertia  ixx="1e-6" ixy="0.0"  ixz="0.0"
+            iyy="1e-6"  iyz="0.0"
+	          izz="1e-6" />
       </inertial>
       <visual>

File: sr_description/hand/xacro/thumb/thbiotac.urdf.xacro (robot description, xacro)
@@ -21,5 +21,7 @@
 	      <mass value="0.016" />
 	      <origin xyz="0 0 0.016" rpy="0 0 0"/>
-	      <inertia  ixx="1" ixy="0.0"  ixz="0.0"  iyy="1"  iyz="0.0" izz="1" />
+	      <inertia  ixx="1e-6" ixy="0.0"  ixz="0.0"
+                  iyy="1e-6"  iyz="0.0"
+                  izz="1e-6" />
       </inertial>
       <visual>

File: sr_description/hand/xacro/thumb/thdistal.urdf.xacro (robot description, xacro)
@@ -12,6 +12,7 @@
 	<mass value="0.016" />
 	<origin xyz="0 0 0.01375" rpy="0 0 0"/>
-	<inertia  ixx="1e-6" ixy="0.0"  ixz="0.0"  iyy="1e-6"  iyz="0.0"
-		  izz="1e-6" />
+	<inertia  ixx="9e-7" ixy="0.0"  ixz="0.0"
+            iyy="9e-7"  iyz="0.0"
+            izz="9e-7" />
       </inertial>
       <visual>
@@ -65,5 +66,7 @@
       <inertial>
 	<mass value="0.001" />
-	<inertia  ixx="0.00001" ixy="0.0"  ixz="0.0"  iyy="0.00001"  iyz="0.0" izz="0.00001" />
+	<inertia  ixx="1e-7" ixy="0.0"  ixz="0.0"
+            iyy="1e-7"  iyz="0.0"
+            izz="1e-7" />
       </inertial>
     </link>

File: sr_description/hand/xacro/thumb/thhub.urdf.xacro (robot description, xacro)
@@ -12,6 +12,7 @@
 	<mass value="0.002" />
 	<origin xyz="0 0 0" rpy="0 0 0"/>
-	<inertia  ixx="1e-6" ixy="0.0"  ixz="0.0"  iyy="1e-6"  iyz="0.0"
-	izz="1e-6" />
+	<inertia  ixx="1e-7" ixy="0.0"  ixz="0.0"
+            iyy="1e-7"  iyz="0.0"
+	          izz="1e-7" />
       </inertial>
       <visual>

File: sr_description/hand/xacro/thumb/thmiddle.urdf.xacro (robot description, xacro)
@@ -12,6 +12,7 @@
 	<mass value="0.016" />
 	<origin xyz="0 0 0.016" rpy="0 0 0"/>
-	<inertia  ixx="1e-6" ixy="0.0"  ixz="0.0"  iyy="1e-6"  iyz="0.0"
-	izz="1e-6" />
+	<inertia  ixx="1e-6" ixy="0.0"  ixz="0.0"
+            iyy="1e-6"  iyz="0.0"
+            izz="1e-6" />
       </inertial>
       <visual>

File: sr_description/hand/xacro/thumb/thproximal.urdf.xacro (robot description, xacro)
@@ -22,5 +22,7 @@
 	<mass value="0.016" />
 	<origin xyz="0 0 0.019" rpy="0 0 0"/>
-	<inertia  ixx="1e-6" ixy="0.0"  ixz="0.0"  iyy="1e-6"  iyz="0.0"	izz="1e-6" />
+	<inertia  ixx="1e-6" ixy="0.0"  ixz="0.0"
+            iyy="1e-6"  iyz="0.0"
+          	izz="1e-6" />
       </inertial>
       <visual>
