Commit message: fix palm inertia

File: sr_description/hand/xacro/palm/palm.urdf.xacro (robot description, xacro)
@@ -22,7 +22,7 @@
 	<origin xyz="0 0 0.035" rpy="0 0 0" />
 	<mass value="0.3" />
-	<inertia  ixx="0.0001" ixy="0.0"  ixz="0.0"
-            iyy="0.0002" iyz="0.0"
-          	izz="0.0001" />
+	<inertia  ixx="0.0000725" ixy="0.0"  ixz="0.0"
+            iyy="0.0001325" iyz="0.0"
+          	izz="0.000185" />
       </inertial>
       <visual>

Commit message: fix palm inertia

File: sr_description/hand/xacro/palm/palm.urdf.xacro (robot description, xacro)
@@ -22,7 +22,7 @@
 	<origin xyz="0 0 0.035" rpy="0 0 0" />
 	<mass value="0.3" />
-	<inertia  ixx="0.0000725" ixy="0.0"  ixz="0.0"
-            iyy="0.0001325" iyz="0.0"
-          	izz="0.000185" />
+	<inertia  ixx="0.0001325" ixy="0.0"  ixz="0.0"
+            iyy="0.000185" iyz="0.0"
+          	izz="0.0000725" />
       </inertial>
       <visual>
